Commit message: 已导入可用的urdf

File: src/arm/model/arm4.urdf (robot description, URDF)
Before this commit: robot arm, 6 links, 5 joints
Links:
- removed link link1
- removed link link2
- removed link link3
- removed link link4
- removed link link5
- added link left1, mass 0.124526845341314; collision mesh filename=package://arm/model//left1.STL; visual mesh filename=package://arm/model//left1.STL
- added link left2, mass 0.0774950388502557; collision mesh filename=package://arm/model//left2.STL; visual mesh filename=package://arm/model//left2.STL
- added link left3, mass 0.0633349973664182; collision mesh filename=package://arm/model//left3.STL; visual mesh filename=package://arm/model//left3.STL
- added link left4, mass 0.0986878737710679; collision mesh filename=package://arm/model//left4.STL; visual mesh filename=package://arm/model//left4.STL
- added link yuntai, mass 0.0552435634534438; collision mesh filename=package://arm/model//yuntai.STL; visual mesh filename=package://arm/model//yuntai.STL
- link base_link: mass 0.013404874825587 -> 0.22839928056115; geometry collision mesh filename=package://arm/model//base_link.STL; visual mesh filename=package://arm/model//base_link.STL
Joints:
- removed joint joint1
- removed joint joint2
- removed joint joint3
- removed joint joint4
- removed joint joint5
- added joint left1: type revolute, parent yuntai, child left1, origin xyz=0.165 -0.00625 0.01 rpy=1.5708 0 3.1416, axis 0 0 1, limit lower=0 upper=0 effort=0 velocity=0
- added joint left2: type revolute, parent left1, child left2, origin xyz=0.14795 0.02 0.00935 rpy=0 0 3.1416, axis 0 0 -1, limit lower=0 upper=0 effort=0 velocity=0
- added joint left3: type revolute, parent left2, child left3, origin xyz=0.213 0 0.0229 rpy=0 0 -1.5708, axis 0 0 1, limit lower=0 upper=0 effort=0 velocity=0
- added joint left4: type fixed, parent left3, child left4, origin xyz=0.1058 0.0275 -0.026 rpy=1.5707963267949 0 0, axis 0 0.720066850328186 0.693904698830066
- added joint yuntai: type revolute, parent base_link, child yuntai, origin xyz=0 0 0.0565 rpy=0 0 0, axis 0 0 -1, limit lower=0 upper=0 effort=0 velocity=0

Commit message: 当前代码是新机械臂代码

File: src/arm/model/arm4.urdf (robot description, URDF)
Before this commit: robot arm, 6 links, 5 joints
Links:
- removed link link1
- removed link link2
- removed link link3
- removed link link4
- removed link link5
- added link joint1, mass 0.0552435634534438; collision mesh filename=package://arm/model/joint1.STL; visual mesh filename=package://arm/model/joint1.STL
- added link joint2, mass 0.124526845341314; collision mesh filename=package://arm/model/joint2.STL; visual mesh filename=package://arm/model/joint2.STL
- added link joint3, mass 0.0774950388502557; collision mesh filename=package://arm/model/joint3.STL; visual mesh filename=package://arm/model/joint3.STL
- added link joint4, mass 0.0633349973664182; collision mesh filename=package://arm/model/joint4.STL; visual mesh filename=package://arm/model/joint4.STL
- added link joint5, mass 0.0986878737710679; collision mesh filename=package://arm/model/joint5.STL; visual mesh filename=package://arm/model/joint5.STL
- link base_link: mass 0.013404874825587 -> 0.22839928056115
Joints:
- joint joint1: child link1 -> joint1; origin xyz=0 0 0.0435 rpy=0 0 0 -> xyz=0 0 0.0565 rpy=0 0 0
- joint joint2: child link2 -> joint2; origin xyz=0.26 0.0162 0.009 rpy=1.5708 0 -3.1416 -> xyz=0.165 -0.00625 0.01 rpy=1.5708 0 3.1416; parent link1 -> joint1
- joint joint3: child link3 -> joint3; origin xyz=0.224 0.0243 -0.0087 rpy=0 0 3.1416 -> xyz=0.14795 0.02 0.00935 rpy=0 0 3.1416; parent link2 -> joint2
- joint joint4: child link4 -> joint4; origin xyz=0.238 -0.0175 0.021 rpy=0 0 -1.5708 -> xyz=0.213 0 0.0229 rpy=0 0 -1.5708; parent link3 -> joint3
- joint joint5: axis 0 0 0 -> 0 0.720066850328186 0.693904698830066; child link5 -> joint5; origin xyz=0.1058 0.0275 -0.026 rpy=3.1416 0 0 -> xyz=0.1058 0.0275 -0.026 rpy=1.5707963267949 0 0; parent link4 -> joint4

Commit message: 将当前的模型的base_link修改为arm_base_link

File: src/arm/model/arm4.urdf (robot description, URDF)
Before this commit: robot arm, 6 links, 5 joints
Links:
- removed link base_link
- added link arm_base_link, mass 0.22839928056115; collision mesh filename=package://arm/model/arm_base_link.STL; visual mesh filename=package://arm/model/arm_base_link.STL
Joints:
- joint joint1: parent base_link -> arm_base_link

Commit message: 初步增加解析解

File: src/arm/model/arm4.urdf (robot description, URDF)
Before this commit: robot arm, 6 links, 5 joints
Joints:
- joint joint1: limit lower=0 upper=0 effort=0 velocity=0 -> lower=-3.15 upper=3.14 effort=10 velocity=10
- joint joint2: limit lower=0 upper=0 effort=0 velocity=0 -> lower=-3.15 upper=3.14 effort=10 velocity=10
- joint joint3: limit lower=0 upper=0 effort=0 velocity=0 -> lower=-3.15 upper=3.14 effort=10 velocity=10
- joint joint4: limit lower=0 upper=0 effort=0 velocity=0 -> lower=-3.15 upper=3.14 effort=10 velocity=10

Commit message: 完善机械臂解析解求解器的多解选择，更新URDF

File: src/arm/model/arm4.urdf (robot description, URDF)
Before this commit: robot arm, 6 links, 5 joints
Links:
- link arm_base_link: mass 0.22839928056115 -> 0.52769
- link joint1: mass 0.0552435634534438 -> 0.055911161682556
- link joint2: mass 0.124526845341314 -> 0.13346
- link joint3: mass 0.0774950388502557 -> 0.085069
- link joint4: mass 0.0633349973664182 -> 0.063335
- link joint5: mass 0.0986878737710679 -> 0.098688
Joints:
- joint joint1: limit lower=-3.15 upper=3.14 effort=10 velocity=10 -> lower=-3.14 upper=3.14 effort=10 velocity=10; origin xyz=0 0 0.0565 rpy=0 0 0 -> xyz=0 0 0.0565000000000001 rpy=0 0 0
- joint joint2: limit lower=-3.15 upper=3.14 effort=10 velocity=10 -> lower=-3.14 upper=3.14 effort=10 velocity=10; origin xyz=0.165 -0.00625 0.01 rpy=1.5708 0 3.1416 -> xyz=0.165000000000001 -0.00624999999999923 0.0099999999999999 rpy=1.5707963267949 0 3.14159265358979
- joint joint3: limit lower=-3.15 upper=3.14 effort=10 velocity=10 -> lower=-3.14 upper=3.14 effort=10 velocity=10; origin xyz=0.14795 0.02 0.00935 rpy=0 0 3.1416 -> xyz=0.19705 0.02 0.00935000000000042 rpy=0 0 3.14159265358979
- joint joint4: limit lower=-3.15 upper=3.14 effort=10 velocity=10 -> lower=-3.14 upper=3.14 effort=10 velocity=10; origin xyz=0.213 0 0.0229 rpy=0 0 -1.5708 -> xyz=0.268 0 0.0228999999999997 rpy=0 0 -1.5707963267949
- joint joint5: axis 0 0.720066850328186 0.693904698830066 -> 0.720066850328186 -0.481503731058444 0.499657770914496; origin xyz=0.1058 0.0275 -0.026 rpy=1.5707963267949 0 0 -> xyz=0.1058 0.0274999999999999 -0.026 rpy=1.5707963267949 0 0

Commit message: 更新机械臂模型

File: src/arm/model/arm4.urdf (robot description, URDF)
Before this commit: robot arm, 6 links, 5 joints
Links:
- link arm_base_link: geometry collision mesh filename=arm_base_link.STL; visual mesh filename=arm_base_link.STL
- link joint1: geometry collision mesh filename=joint1.STL; visual mesh filename=joint1.STL
- link joint2: geometry collision mesh filename=joint2.STL; visual mesh filename=joint2.STL
- link joint3: geometry collision mesh filename=joint3.STL; visual mesh filename=joint3.STL
- link joint4: geometry collision mesh filename=joint4.STL; visual mesh filename=joint4.STL
- link joint5: geometry collision mesh filename=joint5.STL; visual mesh filename=joint5.STL

File: src/arm2/model/arm2.urdf (robot description, URDF)
Before this commit: robot arm2, 6 links, 5 joints
Links:
- link arm_base_link: mass 0.013404874825587 -> 0.530093466980402; geometry collision mesh filename=base_link.STL; visual mesh filename=base_link.STL
- link joint1: mass 0.250946449257902 -> 0.88269255232493; geometry collision mesh filename=link1.STL; visual mesh filename=link1.STL
- link joint2: mass 0.101323280514315 -> 0.253178144050794; geometry collision mesh filename=link2.STL; visual mesh filename=link2.STL
- link joint3: mass 0.060920292136448 -> 0.131053744091016; geometry collision mesh filename=link3.STL; visual mesh filename=link3.STL
- link joint4: mass 0.0555492180755331 -> 0.0735886999783614; geometry collision mesh filename=link4.STL; visual mesh filename=link4.STL
- link joint5: mass 0.0226058648535915 -> 0.098687873771068; geometry collision mesh filename=link5.STL; visual mesh filename=link5.STL
Joints:
- joint joint2: origin xyz=0.26 0.0162 0.009 rpy=1.5708 0 -3.1416 -> xyz=0.260000000000043 0.0162000000000001 0.00900000000008132 rpy=1.5707963267949 0 -3.14159265358979
- joint joint3: axis 0 0 -1 -> 0 0 1; origin xyz=0.224 0.0243 -0.0087 rpy=0 0 3.1416 -> xyz=0.224000000000015 0.0243000000000365 -0.00869999999999983 rpy=3.14159265358979 0 3.14159265358979
- joint joint4: axis 0 0 1 -> 0 0 -1; origin xyz=0.238 -0.0175 0.021 rpy=0 0 -1.5708 -> xyz=0.238000000000014 -0.0175000000000387 0.0360000000000009 rpy=0 0 1.5704
- joint joint5: origin xyz=0.1058 0.0275 -0.026 rpy=3.1416 0 0 -> xyz=0.105799999999993 0.0274999999999227 -0.0259999999999984 rpy=1.5707963267949 1.44388179307632 1.5707963267949

Commit message: 完成URDF的调整

File: src/arm/model/arm4.urdf (robot description, URDF)
Before this commit: robot arm, 6 links, 5 joints
Links:
- link arm_base_link: geometry collision mesh filename=package://arm/model/arm_base_link.STL; visual mesh filename=package://arm/model/arm_base_link.STL
- link joint1: geometry collision mesh filename=package://arm/model/joint1.STL; visual mesh filename=package://arm/model/joint1.STL
- link joint2: geometry collision mesh filename=package://arm/model/joint2.STL; visual mesh filename=package://arm/model/joint2.STL
- link joint3: geometry collision mesh filename=package://arm/model/joint3.STL; visual mesh filename=package://arm/model/joint3.STL
- link joint4: geometry collision mesh filename=package://arm/model/joint4.STL; visual mesh filename=package://arm/model/joint4.STL
- link joint5: geometry collision mesh filename=package://arm/model/joint5.STL; visual mesh filename=package://arm/model/joint5.STL

File: src/arm2/model/arm2.urdf (robot description, URDF)
Before this commit: robot arm2, 6 links, 5 joints
Links:
- link arm_base_link: mass 0.530093466980402 -> 0.66509; geometry collision mesh filename=package://arm2/model/base_link.STL; visual mesh filename=package://arm2/model/base_link.STL
- link joint1: mass 0.88269255232493 -> 0.27086; geometry collision mesh filename=package://arm2/model/link1.STL; visual mesh filename=package://arm2/model/link1.STL
- link joint2: mass 0.253178144050794 -> 0.11716; geometry collision mesh filename=package://arm2/model/link2.STL; visual mesh filename=package://arm2/model/link2.STL
- link joint3: mass 0.131053744091016 -> 0.13105; geometry collision mesh filename=package://arm2/model/link3.STL; visual mesh filename=package://arm2/model/link3.STL
- link joint4: mass 0.0735886999783614 -> 0.039471; geometry collision mesh filename=package://arm2/model/link4.STL; visual mesh filename=package://arm2/model/link4.STL
- link joint5: mass 0.098687873771068 -> 0.098688; geometry collision mesh filename=package://arm2/model/link5.STL; visual mesh filename=package://arm2/model/link5.STL
Joints:
- joint joint1: origin xyz=0 0 0.0435 rpy=0 0 0 -> xyz=0 0 0.045 rpy=0 0 0
- joint joint2: origin xyz=0.260000000000043 0.0162000000000001 0.00900000000008132 rpy=1.5707963267949 0 -3.14159265358979 -> xyz=0.26 0.0162 0.0075 rpy=1.5708 0 -3.1416
- joint joint3: axis 0 0 1 -> 0 0 -1; origin xyz=0.224000000000015 0.0243000000000365 -0.00869999999999983 rpy=3.14159265358979 0 3.14159265358979 -> xyz=0.224 0.0243 0.0237 rpy=0 0 3.1415
- joint joint4: origin xyz=0.238000000000014 -0.0175000000000387 0.0360000000000009 rpy=0 0 1.5704 -> xyz=0.238 0.0175 -0.021 rpy=0 0 -1.5704
- joint joint5: origin xyz=0.105799999999993 0.0274999999999227 -0.0259999999999984 rpy=1.5707963267949 1.44388179307632 1.5707963267949 -> xyz=0.1058 -0.0275 0.026 rpy=1.5708 0 0
