Commit message: 修改机械臂模型

File: src/arm/model/arm4.urdf (robot description, URDF)
Before this commit: robot arm, 6 links, 5 joints
Links:
- link arm_base_link: mass 0.52769 -> 0.527622512880337
- link joint1: mass 0.055911161682556 -> 0.127701870541598
- link joint2: mass 0.13346 -> 0.245916230331252
- link joint3: mass 0.085069 -> 0.134998289963193
- link joint4: mass 0.063335 -> 0.0613085781646441
- link joint5: mass 0.098688 -> 0.0986878737710681
Joints:
- joint joint2: origin xyz=0.165000000000001 -0.00624999999999923 0.0099999999999999 rpy=1.5707963267949 0 3.14159265358979 -> xyz=0.165000000000001 0.00670000000000074 0.0100000000000004 rpy=1.5707963267949 0 -3.14159265358979
- joint joint3: axis 0 0 -1 -> 0 0 1; origin xyz=0.19705 0.02 0.00935000000000042 rpy=0 0 3.14159265358979 -> xyz=0.209 0.0242999999999992 -0.00169999999999987 rpy=-3.14159265358979 0 3.14159265358979
- joint joint4: origin xyz=0.268 0 0.0228999999999997 rpy=0 0 -1.5707963267949 -> xyz=0.237999999999993 0.0174999999999935 -0.0209999999999999 rpy=-3.14159265358979 0 1.5707963267949
- joint joint5: origin xyz=0.1058 0.0274999999999999 -0.026 rpy=1.5707963267949 0 0 -> xyz=0.1058 0.0274999999999999 -0.0259999999999996 rpy=1.5707963267949 0 0
